File: UINIO-Peg-Board.kicad_pcb (KiCad board)
At the start: 2 copper layers, 100 x 100 mm, 0 parts

Commit message: Generate Gerber files.
Other:
- board text removed: "N0. 1"

Commit message: Generate Gerber files.
Other:
- board text added: "Version 0.0.1"

Commit message: Release UINIO-Peg-Board version 0.0.1.
Other:
- board text added: "UINIO-Peg-Board"

Commit message: Release UINIO-Peg-Board version 1.0.0.
Other:
- board text added: "Version 1.0.0"
- board text removed: "Version 0.0.1"

Commit message: Release UINIO-Peg-Board version 1.0.1.
Other:
- board text added: "Version 1.0.1"
- board text removed: "Version 1.0.0"
